File: Thinkpad700CPower.kicad_sch (KiCad schematic)
At the start: 368 parts, among them CN1 AC_ADAPT, CN2 BATT, CN3 stdby_bat, CN4 TO_MB, CN5 LCD_PWR, IC1 unknown, IC11 uPC1100G, IC12 uPC1100G, IC3 "4A" "31", IC4 LM324, IC5 LM324, IC6 LM2903, J1 0, Q1 2SJ189, Q10 "L6", Q11 2SA1213?, Q12 2SJ246, Q13 "26", Q14 2SA1203, Q15 "94", Q16 2SJ189, Q17 2SD1368?, Q18 2SA1947?, Q19 "AB" "TN", Q2 2SJ189, Q20 "AB" "TN", Q200 "L6", Q201 "L6", Q21 2SC4213, Q24 "G16" 2SK1590, Q25 2SC4213, Q26 "G16" 2SK1590, Q27 DTA114, Q29 2SA1213?, Q3 DTC144EUB, Q30 2SD1368, Q300 EE 3N ???, Q301 "G16" 2SK1590, Q302 "ZS", Q303 "L6", Q304 "M6" 2SA1611, Q305 "G16" 2SK1590, Q306 "26", Q307 2SA1411 "M15", Q308 2SA1411 "M15", Q309 "M15", Q31 2SJ182, Q310 "26", Q311 EMG1 "G1", Q32 2SK2463, Q33 2SK2463, Q34 "96", Q35 "M15", Q36 "G16" 2SK1590, Q4 2SA1213?, Q40 "ZS", Q41 "G16" 2SK1590, Q42 "16", Q45 "16", Q47 2SC4213, Q48 2SK974, Q5 "L6", Q51 "O4", Q52 2SJ189, Q53 2SK1469, Q54 2SK1469, Q56 2SK974, Q59 EMG2 "G2", Q6 2SJ189, Q60 "M6" 2SA1611, Q61 "O4", Q62 "M6" 2SA1611, Q63 "O4", Q64 "M6" 2SA1611, Q65 "O4", Q66 "26", Q67 "NY", Q68 2SK1590 "G16", Q7 2SJ189, Q9 2SC4213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

Commit message: update voltage rail names
Parts:
- D14: value 1.2V? (122) -> "122" 12V
- D19: value "162" -> "162" 16V
- D4: value 1.01V? (101) -> "101" 10V?
- D5: value 5.2? (512) -> "512" 5.1V?
Connections:
- net VQUESTION renamed +5VD
- net VREF renamed VREF_2V5
- net VREF_2V5: now also C23.2, IC3.1 (Pin_1), R67.1, VR5.2
- net VREF2 renamed VREF_5V0
- net VREF_5V0: no longer C23.2, IC3.1 (Pin_1), R67.1, VR5.2
- net VREF_IC12_2V5 renamed VREF_2V5_IC12_2V5
- net negative_rail renamed -5V
- net negative_rail_sw renamed N5V_SW
- net negative_rail_sw2 renamed N5V_SW2
- net positive_rail renamed +3V8
- net positive_rail_sw renamed 3V8_SW
Other:
- note added: "comparator supply (about 6.7V)"
- note removed: "5V analog ref"
- note removed: "comparator supply"
