File: 700CPowerBoard/Thinkpad700CPower.kicad_sch (KiCad schematic)
At the start: 409 parts, among them CN1 AC_ADAPT, CN10 BATT, CN2 BATT, CN3 stdby_bat, CN4 TO_MB, CN5 LCD_PWR, IC1 DT 2Y (SOT-89), IC11 uPC1100G, IC12 uPC1100G, IC3 "4A" "31", IC4 LM324, IC5 LM324, IC6 LM2903, J1 0, Q1 2SJ189, Q10 "L6", Q11 2SA1213?, Q12 2SJ246, Q13 "26", Q14 2SA1203, Q15 "94", Q16 2SJ189, Q17 2SD1368?, Q18 2SA1947?, Q19 "AB" "TN", Q2 2SJ189, Q20 "AB" "TN", Q200 "L6", Q201 "L6", Q21 2SC4213, Q24 "G16" 2SK1590, Q25 2SC4213, Q26 "G16" 2SK1590, Q27 DTA114, Q29 2SA1213?, Q3 DTC144EUB, Q30 2SD1368, Q300 EE 3N (SOT-89), Q301 "G16" 2SK1590, Q302 "ZS", Q303 "L6", Q304 2SA1611 "M6", Q305 "G16" 2SK1590, Q306 "26", Q307 2SA1411 "M15", Q308 2SA1411(M15), Q309 "M15", Q31 2SJ182, Q310 "26", Q311 EMG1 "G1", Q32 2SK2463, Q33 2SK2463, Q34 "96", Q35 "M15", Q36 2SK1590, Q4 2SA1213?, Q40 "ZS", Q41 "G16" 2SK1590, Q42 "16", Q45 "16", Q47 2SC4213, Q48 2SK974, Q5 "L6", Q51 "O4", Q52 2SJ189, Q53 2SK1469, Q54 2SK1469, Q56 2SK974, Q59 EMG2 "G2", Q6 2SJ189, Q60 "M6" 2SA1611, Q61 "O4", Q62 "M6" 2SA1611, Q63 "O4", Q64 "M6" 2SA1611, Q65 "O4", Q66 "26", Q67 "NY", Q68 2SK1590 "G16", Q7 2SJ189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

Commit message: Add info on external battery current sense
Parts:
- added R9: 15mOhm, symbol Device:R_Small_US
Connections:
- net at BT18.2 (-), CN10.6 (Pin_6), TH10.1: now also R9.1; no longer BT3.2 (-), CN10.3 (Pin_3), CN10.4 (Pin_4)
- net CN2_4 renamed BAT_CS1
- net CN2_6 renamed BAT_CS2
- net CN4_14 renamed CURSENSE/~{ZERO}
- net IC4_8_OUT renamed PACK_ISENSE
- new net: BT3.2 (-), CN10.3 (Pin_3), CN10.4 (Pin_4), R9.2
Other:
- note added: "Current sense in external battery pack"
- note added: "Mux for CS amp Zero-out function (offset compensation)"
- note added: "V=0.15*Ibatt/2 + 2.5"
- note removed: "Cell monitoring Cell balancing?"
- moved on the sheet: R81
